File: kicad-blind-burried-vias.kicad_pcb (KiCad board)
At the start: 6 copper layers, 62 x 53 mm, 2 parts

Commit message: Add burried VIA (In1.Cu-In4.CU), End-Start and Connected layers
Routing:
- net /blind_vias_path: track 52.4 -> 76.1 mm, vias 2 -> 3
Changed lines of the file:
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@@
   (segment (start 143.745 112.245) (end 153.345 112.245) (width 0.25) (layer "In1.Cu") (net 1))
   (segment (start 153.6 111.99) (end 153.6 109.2) (width 0.25) (layer "In1.Cu") (net 1))
+  (segment (start 153.6 109.2) (end 153.6 107.3) (width 0.25) (layer "In1.Cu") (net 1))
+  (via blind (at 153.6 107.3) (size 0.8) (drill 0.4) (layers "In1.Cu" "In4.Cu") (remove_unused_layers) (keep_end_layers) (net 1))
   (via blind (at 153.6 109.2) (size 0.8) (drill 0.4) (layers "In1.Cu" "In2.Cu") (net 1))
+  (segment (start 158.6 109.2) (end 165.955 109.2) (width 0.25) (layer "In2.Cu") (net 1))
   (segment (start 165.955 109.2) (end 169 112.245) (width 0.25) (layer "In2.Cu") (net 1))
-  (segment (start 153.6 109.2) (end 165.955 109.2) (width 0.25) (layer "In2.Cu") (net 1))
+  (segment (start 153.6 109.2) (end 158.6 109.2) (width 0.25) (layer "In2.Cu") (net 1))
+  (segment (start 153.6 107.3) (end 150.7 107.3) (width 0.25) (layer "In3.Cu") (net 1))
+  (segment (start 153.6 107.3) (end 166.5275 107.3) (width 0.25) (layer "In4.Cu") (net 1))
+  (segment (start 166.5275 107.3) (end 169 109.7725) (width 0.25) (layer "In4.Cu") (net 1))
+  (segment (start 169 109.7725) (end 169 112.245) (width 0.25) (layer "In4.Cu") (net 1))
   (segment (start 136.47 81.765) (end 151.535 81.765) (width 0.25) (layer "F.Cu") (net 2))
   (segment (start 151.535 81.765) (end 151.6 81.7) (width 0.25) (layer "F.Cu") (net 2))

Commit message: Add burried VIA (In1.Cu-In4.CU), Connected layers only
Routing:
- net /blind_vias_path: track 76.1 -> 100.2 mm, vias 3 -> 4
Changed lines of the file:
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@@
   (segment (start 143.7 112.2) (end 143.745 112.245) (width 0.25) (layer "In1.Cu") (net 1))
   (segment (start 153.345 112.245) (end 169 112.245) (width 0.25) (layer "In1.Cu") (net 1))
+  (segment (start 153.6 107.3) (end 153.6 105.5) (width 0.25) (layer "In1.Cu") (net 1))
   (segment (start 143.745 112.245) (end 153.345 112.245) (width 0.25) (layer "In1.Cu") (net 1))
   (segment (start 153.6 111.99) (end 153.6 109.2) (width 0.25) (layer "In1.Cu") (net 1))
@@
   (via blind (at 153.6 107.3) (size 0.8) (drill 0.4) (layers "In1.Cu" "In4.Cu") (remove_unused_layers) (keep_end_layers) (net 1))
   (via blind (at 153.6 109.2) (size 0.8) (drill 0.4) (layers "In1.Cu" "In2.Cu") (net 1))
+  (via blind (at 153.6 105.5) (size 0.8) (drill 0.4) (layers "In1.Cu" "In4.Cu") (remove_unused_layers) (net 1))
   (segment (start 158.6 109.2) (end 165.955 109.2) (width 0.25) (layer "In2.Cu") (net 1))
   (segment (start 165.955 109.2) (end 169 112.245) (width 0.25) (layer "In2.Cu") (net 1))
   (segment (start 153.6 109.2) (end 158.6 109.2) (width 0.25) (layer "In2.Cu") (net 1))
+  (segment (start 170.4 110.845) (end 169 112.245) (width 0.25) (layer "In3.Cu") (net 1))
+  (segment (start 167.4 105.5) (end 170.4 108.5) (width 0.25) (layer "In3.Cu") (net 1))
+  (segment (start 153.6 105.5) (end 167.4 105.5) (width 0.25) (layer "In3.Cu") (net 1))
   (segment (start 153.6 107.3) (end 150.7 107.3) (width 0.25) (layer "In3.Cu") (net 1))
+  (segment (start 170.4 108.5) (end 170.4 110.845) (width 0.25) (layer "In3.Cu") (net 1))
   (segment (start 153.6 107.3) (end 166.5275 107.3) (width 0.25) (layer "In4.Cu") (net 1))
   (segment (start 166.5275 107.3) (end 169 109.7725) (width 0.25) (layer "In4.Cu") (net 1))
